File: hardware/V1_revB/0_ramn/ramn.kicad_pcb (KiCad board)
At the start: 2 copper layers, 85.6 x 54 mm, 106 parts, among them J1 USB_C_Micro, J2 Screw_Terminal_01x03, J3 , J4 , J5 , J6 , U1 ATA6561-GAQW-N, U10 ATA6561-GAQW-N, U11 STM32L443CCTx, U12 NCV8163, U2 STM32L443CCTx, U3 NCV8163, U4 ATA6561-GAQW-N, U5 STM32L443CCTx, U6 NCV8163, U7 ATA6561-GAQW-N, U8 STM32L443CCTx, U9 NCV8163, Y1 NX3225GD-8MHZ-STD-CRA-3, Y2 NX3225GD-8MHZ-STD-CRA-3, Y3 NX3225GD-8MHZ-STD-CRA-3, Y4 NX3225GD-8MHZ-STD-CRA-3

Commit message: feat (hw): change USB to USB C and change Test points footprints
Parts:
- removed J1: USB_C_Micro, Connector_USB:USB_Micro-B_Wuerth_629105150521
- removed RX, TX: , TestPoint:TestPoint_Pad_D1.0mm
- added P1: USB_C_Plug_USB2.0, Library:C393939, F.Cu at (45.9, 59.3)
- added R18: 5k1, Resistor_SMD:R_0603_1608Metric, F.Cu at (49.9, 57.5)
- added R19: 5k1, Resistor_SMD:R_0603_1608Metric, F.Cu at (49.1, 61.0)
- added RX1: , TestPoint:TestPoint_Pad_D1.0mm, F.Cu at (106.7, 61.6)
- added TX1: , TestPoint:TestPoint_Pad_D1.0mm, F.Cu at (106.7, 58.4)
- R8: value DNM -> 10k
- R9: value 10k -> DNM
- TP1, TP10, TP2, TP3, TP4, TP5, TP6, TP7, TP8, TP9: footprint TestPoint:TestPoint_Loop_D2.54mm_Drill1.5mm_Beaded -> Global_Library:KEYSTONE_5002
- U11, U2, U5, U8: value STM32L443CCTx -> STM32L552/STM32L562
Connections:
- net /usb_uc/ECU_1_EN renamed /ECUB/ECU_ENABLE
- net /usb_uc/ECU_2_EN renamed /ECUC/ECU_ENABLE
- net /usb_uc/ECU_3_EN renamed /ECUD/ECU_ENABLE
- C35 pad 1: Net-(C35-Pad1) -> Net-(U11-PH0)
- R1 pad 2: Net-(J1-Pad1) -> Net-(P1-VBUS-PadA4)
- U11 pad 10: Net-(U11-Pad10) -> unconnected-(U11-PA0-Pad10)
- U11 pad 2: Net-(U11-Pad2) -> unconnected-(U11-PC13-Pad2)
- U11 pad 30: Net-(U11-Pad30) -> unconnected-(U11-PA9-Pad30)
- U11 pad 31: Net-(U11-Pad31) -> unconnected-(U11-PA10-Pad31)
- U11 pad 32: Net-(U11-Pad32) -> unconnected-(U11-PA11-Pad32)
- U11 pad 33: Net-(U11-Pad33) -> unconnected-(U11-PA12-Pad33)
- U11 pad 4: Net-(U11-Pad4) -> unconnected-(U11-PC15-Pad4)
- U11 pad 41: Net-(U11-Pad41) -> unconnected-(U11-PB5-Pad41)
- U11 pad 42: Net-(U11-Pad42) -> unconnected-(U11-PB6-Pad42)
- U11 pad 43: Net-(U11-Pad43) -> unconnected-(U11-PB7-Pad43)
- U11 pad 5: Net-(C35-Pad1) -> Net-(U11-PH0)
- U12 pad 4: Net-(U12-Pad4) -> unconnected-(U12-NC-Pad4)
- U2 pad 30: Net-(U2-Pad30) -> unconnected-(U2-PA9-Pad30)
- U2 pad 31: Net-(U2-Pad31) -> unconnected-(U2-PA10-Pad31)
- U3 pad 4: Net-(U3-Pad4) -> unconnected-(U3-NC-Pad4)
- U5 pad 10: Net-(U5-Pad10) -> unconnected-(U5-PA0-Pad10)
- U5 pad 2: Net-(U5-Pad2) -> unconnected-(U5-PC13-Pad2)
- U5 pad 30: Net-(U5-Pad30) -> unconnected-(U5-PA9-Pad30)
- U5 pad 31: Net-(U5-Pad31) -> unconnected-(U5-PA10-Pad31)
- U5 pad 32: Net-(U5-Pad32) -> unconnected-(U5-PA11-Pad32)
- U5 pad 33: Net-(U5-Pad33) -> unconnected-(U5-PA12-Pad33)
- U5 pad 4: Net-(U5-Pad4) -> unconnected-(U5-PC15-Pad4)
- U5 pad 41: Net-(U5-Pad41) -> unconnected-(U5-PB5-Pad41)
- U5 pad 42: Net-(U5-Pad42) -> unconnected-(U5-PB6-Pad42)
- U5 pad 43: Net-(U5-Pad43) -> unconnected-(U5-PB7-Pad43)
- U6 pad 4: Net-(U6-Pad4) -> unconnected-(U6-NC-Pad4)
- U8 pad 10: Net-(U8-Pad10) -> unconnected-(U8-PA0-Pad10)
- U8 pad 2: Net-(U8-Pad2) -> unconnected-(U8-PC13-Pad2)
- U8 pad 30: Net-(U8-Pad30) -> unconnected-(U8-PA9-Pad30)
- U8 pad 31: Net-(U8-Pad31) -> unconnected-(U8-PA10-Pad31)
- U8 pad 32: Net-(U8-Pad32) -> unconnected-(U8-PA11-Pad32)
- U8 pad 33: Net-(U8-Pad33) -> unconnected-(U8-PA12-Pad33)
- U8 pad 4: Net-(U8-Pad4) -> unconnected-(U8-PC15-Pad4)
- U8 pad 41: Net-(U8-Pad41) -> unconnected-(U8-PB5-Pad41)
- U8 pad 42: Net-(U8-Pad42) -> unconnected-(U8-PB6-Pad42)
- U8 pad 43: Net-(U8-Pad43) -> unconnected-(U8-PB7-Pad43)
- U9 pad 4: Net-(U9-Pad4) -> unconnected-(U9-NC-Pad4)
- Y4 pad 1: Net-(C35-Pad1) -> Net-(U11-PH0)
Routing:
- net GND: track 332.8 -> 356.1 mm, vias 121 -> 130
- net Net-(P1-VBUS-PadA4): track 0.00 -> 20.4 mm
- net Net-(U11-PH0): track 0.00 -> 17.6 mm
- net Net-(C35-Pad1): track 17.6 -> 0.00 mm
- net Net-(J1-Pad1): track 15.6 -> 0.00 mm
- net Net-(P1-SHIELD): track 15.4 -> 28.0 mm
- net Net-(P1-VCONN): track 0.00 -> 2.80 mm
- net /usb_uc/USB_D+: track 7.28 -> 9.97 mm
- net Net-(P1-CC): track 0.00 -> 2.66 mm
- net /usb_uc/USB_D-: track 7.33 -> 9.95 mm
- net /usb_uc/SYS_JTRST: track 40.6 -> 43.1 mm
- net /usb_uc/BOOT0: track 35.3 -> 36.4 mm
- net /usb_uc/3V3_ECU: track 99.2 -> 100.2 mm
Other:
- net class 3V removed
- net class 5V removed
- net class CAN removed
- net class Default removed
