File: hardware/V1_revB/0_ramn/ramn.kicad_sch (KiCad schematic)
At the start: 29 parts, among them J2 Screw_Terminal_01x03, P1 USB_C_Plug_USB2.0

Commit message: Feat(Hw):Modify_BOM_LCSC#
Parts:
- C1, C2: LCSC# (none) -> C335546
- C43: LCSC# (none) -> C599645
- J2: LCSC# (none) -> C5443579
- R1, R4, R5: LCSC# (none) -> C95177
- R17: LCSC# (none) -> C98220
- R2, R3, R6, R7: LCSC# (none) -> C23090
- TP1, TP2, TP3, TP4, TP5, TP6, TP7: value (none) -> (none); LCSC# (none) -> C5277086

Commit message: Feat(Hw): Modify_and_fix_footprints_and_symbols
Parts:
- FID1, FID2, FID3, H1, H2, H3, H4: now not fitted
Changed lines of the file:
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@@
 		(on_board yes)
 		(in_pos_files yes)
-		(dnp no)
+		(dnp yes)
 		(property "Reference" "H1"
 			(at 29.21 141.0716 0)
@@
 		(on_board yes)
 		(in_pos_files yes)
-		(dnp no)
+		(dnp yes)
 		(property "Reference" "H3"
 			(at 50.8 141.0716 0)
@@
 		(on_board yes)
 		(in_pos_files yes)
-		(dnp no)
+		(dnp yes)
 		(property "Reference" "H2"
 			(at 29.21 151.2316 0)
@@
 		(on_board yes)
 		(in_pos_files yes)
-		(dnp no)
+		(dnp yes)
 		(property "Reference" "H4"
 			(at 50.8 151.2316 0)
@@
 		(on_board yes)
 		(in_pos_files yes)
-		(dnp no)
+		(dnp yes)
 		(property "Reference" "FID1"
 			(at 28.829 162.6616 0)
@@
 		(on_board yes)
 		(in_pos_files yes)
-		(dnp no)
+		(dnp yes)
 		(property "Reference" "FID2"
 			(at 42.799 162.6616 0)
@@
 		(on_board yes)
 		(in_pos_files yes)
-		(dnp no)
+		(dnp yes)
 		(property "Reference" "FID3"
 			(at 56.769 162.6616 0)
@@
 					(unit 1)
 				)
-				(path "/5c9d0d4a-249f-45d4-a492-4d8f074d1b1c/00000000-0000-0000-0000-00005d815e09"
-					(reference "R?")
-					(unit 1)
-				)
-				(path "/5c9d0d4a-249f-45d4-a492-4d8f074d1b1c/00000000-0000-0000-0000-00005d8ede42"
-					(reference "R?")
-					(unit 1)
-				)
 			)
 		)
@@
 					(unit 1)
 				)
-				(path "/5c9d0d4a-249f-45d4-a492-4d8f074d1b1c/00000000-0000-0000-0000-00005d815e09"
-					(reference "C?")
-					(unit 1)
-				)
-				(path "/5c9d0d4a-249f-45d4-a492-4d8f074d1b1c/00000000-0000-0000-0000-00005d8bffce"
-					(reference "C?")
-					(unit 1)
-				)
-				(path "/5c9d0d4a-249f-45d4-a492-4d8f074d1b1c/00000000-0000-0000-0000-00005d8ede42"
-					(reference "C?")
-					(unit 1)
-				)

Commit message: Feat(Hw): UpdateKiCadProjectAndStandardizeComponentProperties
Parts:
- C1, C2: Category (none) -> Electronic Components / Capacitors; LCSC# C335546 -> (none); lcsc# (none) -> C335546; manf# (none) -> 0603B472K250CT
- C43: Category (none) -> Electronic Components / Capacitors; LCSC# C599645 -> (none); lcsc# (none) -> C599645; manf# (none) -> C0603C104J3RAC7867
- FID1, FID2, FID3: Category (none) -> Electronic Components / Other Components
- H1, H2, H3, H4: Category (none) -> Production & Packaging / Screws & Hardware
- J2: Category (none) -> Electronic Components / Connectors; LCSC# C5443579 -> (none); lcsc# (none) -> C5443579; manf# (none) -> 1770966
- P1: Category (none) -> Electronic Components / Connectors; LCSC# C393939 -> (none); lcsc# (none) -> C393939
- R1, R4, R5: Category (none) -> Electronic Components / Resistors; LCSC# C95177 -> (none); lcsc# (none) -> C95177; manf# (none) -> RC0603JR-070RL
- R17: Category (none) -> Electronic Components / Resistors; LCSC# C98220 -> (none); lcsc# (none) -> C98220; manf# (none) -> RC0603FR-0710KL
- R18, R19: Category (none) -> Electronic Components / Resistors; LCSC# C191782 -> (none); lcsc# (none) -> C191782
- R2, R3, R6, R7: Category (none) -> Electronic Components / Resistors; LCSC# C23090 -> (none); lcsc# (none) -> C23090; manf# (none) -> 0603WAF604JT5E
- TP1, TP2, TP3, TP4, TP5, TP6, TP7: value (none) -> ~; Category (none) -> Electronic Components / Other Components; LCSC# C5277086 -> (none); lcsc# (none) -> C5277086; manf# (none) -> RH-5000
