File: hardware/V1_revB/0_ramn/sc_uc.kicad_sch (KiCad schematic)
At the start: 20 parts, among them J6 , U10 ATA6561-GAQW-N

Commit message: Feat(Hw):Modify_BOM_LCSC#
Parts:
- C33, C34, C38, C39, C40: renamed from C?; LCSC# (none) -> C599645
- C35, C36: renamed from C?; LCSC# (none) -> C9807
- C37: renamed from C?; LCSC# (none) -> C1848
- J6: value (none) -> (none); LCSC# (none) -> C2897414
- R14, R15: renamed from R?; LCSC# (none) -> C98220
- R16: renamed from R?; LCSC# (none) -> C95177
- RX1: renamed from RX?; value (none) -> (none); LCSC# (none) -> C5277086
- TP10, TP8, TP9: renamed from TP?; value (none) -> (none); LCSC# (none) -> C5277086
- TX1: renamed from TX?; value (none) -> (none); LCSC# (none) -> C5277086
- U10: LCSC# (none) -> C124015
- U11: renamed from U?; LCSC# (none) -> C2969980
- Y4: renamed from Y?; LCSC# (none) -> C889706

Commit message: Feat(Hw): UpdateKiCadProjectAndStandardizeComponentProperties
Parts:
- C33, C34, C38, C39, C40: Category (none) -> Electronic Components / Capacitors; LCSC# C599645 -> (none); lcsc# (none) -> C599645; manf# (none) -> C0603C104J3RAC7867
- C35, C36: Category (none) -> Electronic Components / Capacitors; LCSC# C9807 -> (none); lcsc# (none) -> C9807; manf# (none) -> CL31A106KAHNNNE
- C37: Category (none) -> Electronic Components / Capacitors; LCSC# C1848 -> (none); lcsc# (none) -> C1848; manf# (none) -> CL31B105KBHNNNE
- J6: value (none) -> ~; Category (none) -> Electronic Components / Connectors; LCSC# C2897414 -> (none); lcsc# (none) -> C2897414; manf# (none) -> PM254-2-13-Z-8.5
- R14, R15: Category (none) -> Electronic Components / Resistors; LCSC# C98220 -> (none); lcsc# (none) -> C98220; manf# (none) -> RC0603FR-0710KL
- R16: Category (none) -> Electronic Components / Resistors; LCSC# C95177 -> (none); lcsc# (none) -> C95177; manf# (none) -> RC0603JR-070RL
- RX1, TX1: value (none) -> ~; Category (none) -> Electronic Components / Switches; LCSC# C5277086 -> (none); lcsc# (none) -> C5277086; manf# (none) -> RH-5000
- TP10, TP8, TP9: value (none) -> ~; Category (none) -> Electronic Components / Other Components; LCSC# C5277086 -> (none); lcsc# (none) -> C5277086; manf# (none) -> RH-5000
- U10: Category (none) -> Electronic Components / Integrated Circuits; LCSC# C124015 -> (none); lcsc# (none) -> C124015; manf# (none) -> MCP2558FD-H/SN
- U11: Category (none) -> Electronic Components / Integrated Circuits; LCSC# C2969980 -> (none); lcsc# (none) -> C2969980; manf# (none) -> STM32L552CET6
- Y4: Category (none) -> Electronic Components / Crystals & Oscillators; LCSC# C889706 -> (none); lcsc# (none) -> C889706; manf# (none) -> NX3225GD-8MHZ-STD-CRA-3
