File: hardware/V1_revB/0_ramn/usb_uc.kicad_sch (KiCad schematic)
At the start: 15 parts, among them U1 ATA6561-GAQW-N

Commit message: Feat(Hw):Modify_BOM_LCSC#
Parts:
- BOOT0: renamed from BOOT?; value (none) -> (none); LCSC# (none) -> C5277086
- C10, C3, C4, C8, C9: renamed from C?; LCSC# (none) -> C599645
- C5, C6: renamed from C?; LCSC# (none) -> C9807
- C7: renamed from C?; LCSC# (none) -> C1848
- J3: renamed from J?; value (none) -> (none); LCSC# (none) -> C2897414
- R8: renamed from R?; LCSC# (none) -> C98220
- U1: LCSC# (none) -> C124015
- U2: renamed from U?; LCSC# (none) -> C2969980
- Y1: renamed from Y?; LCSC# (none) -> C889706
- gave numbers to parts that had none: 1

Commit message: Feat(Hw): Modify_and_fix_footprints_and_symbols
Parts:
- R9: now not fitted
Changed lines of the file:
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@@
 		(instances
 			(project "ramn"
-				(path "/5c9d0d4a-249f-45d4-a492-4d8f074d1b1c"
-					(reference "#PWR?")
-					(unit 1)
-				)
-				(path "/5c9d0d4a-249f-45d4-a492-4d8f074d1b1c/00000000-0000-0000-0000-00005d815e09"
-					(reference "#PWR?")
-					(unit 1)
-				)
 				(path "/5c9d0d4a-249f-45d4-a492-4d8f074d1b1c/00000000-0000-0000-0000-00005d8bffce"
 					(reference "#PWR012")
-					(unit 1)
-				)
-				(path "/5c9d0d4a-249f-45d4-a492-4d8f074d1b1c/00000000-0000-0000-0000-00005d8ede42"
-					(reference "#PWR?")
 					(unit 1)
 				)
@@
 		(instances
 			(project "ramn"
-				(path "/5c9d0d4a-249f-45d4-a492-4d8f074d1b1c/00000000-0000-0000-0000-00005d7dea89"
-					(reference "#PWR?")
-					(unit 1)
-				)
-				(path "/5c9d0d4a-249f-45d4-a492-4d8f074d1b1c/00000000-0000-0000-0000-00005d815e09"
-					(reference "#PWR?")
-					(unit 1)
-				)
 				(path "/5c9d0d4a-249f-45d4-a492-4d8f074d1b1c/00000000-0000-0000-0000-00005d8bffce"
 					(reference "#PWR011")
-					(unit 1)
-				)
-				(path "/5c9d0d4a-249f-45d4-a492-4d8f074d1b1c/00000000-0000-0000-0000-00005d8ede42"
-					(reference "#PWR?")
 					(unit 1)
 				)
@@
 		(instances
 			(project "ramn"
-				(path "/5c9d0d4a-249f-45d4-a492-4d8f074d1b1c"
-					(reference "U?")
-					(unit 1)
-				)
 				(path "/5c9d0d4a-249f-45d4-a492-4d8f074d1b1c/00000000-0000-0000-0000-00005d8bffce"
 					(reference "U2")
@@
 		(instances
 			(project "ramn"
-				(path "/5c9d0d4a-249f-45d4-a492-4d8f074d1b1c"
-					(reference "C?")
-					(unit 1)
-				)
 				(path "/5c9d0d4a-249f-45d4-a492-4d8f074d1b1c/00000000-0000-0000-0000-00005d8bffce"
 					(reference "C9")
@@
 		(instances
 			(project "ramn"
-				(path "/5c9d0d4a-249f-45d4-a492-4d8f074d1b1c"
-					(reference "C?")
-					(unit 1)
-				)
 				(path "/5c9d0d4a-249f-45d4-a492-4d8f074d1b1c/00000000-0000-0000-0000-00005d8bffce"
 					(reference "C10")
@@
 		(instances
 			(project "ramn"
-				(path "/5c9d0d4a-249f-45d4-a492-4d8f074d1b1c"
-					(reference "#PWR?")
-					(unit 1)
-				)
 				(path "/5c9d0d4a-249f-45d4-a492-4d8f074d1b1c/00000000-0000-0000-0000-00005d8bffce"
 					(reference "#PWR019")
@@
 		(instances
 			(project "ramn"
-				(path "/5c9d0d4a-249f-45d4-a492-4d8f074d1b1c"
-					(reference "#PWR?")
-					(unit 1)
-				)
 				(path "/5c9d0d4a-249f-45d4-a492-4d8f074d1b1c/00000000-0000-0000-0000-00005d8bffce"
 					(reference "#PWR018")
@@
 		(instances
 			(project "ramn"
-				(path "/5c9d0d4a-249f-45d4-a492-4d8f074d1b1c"
-					(reference "#PWR?")
-					(unit 1)
-				)
 				(path "/5c9d0d4a-249f-45d4-a492-4d8f074d1b1c/00000000-0000-0000-0000-00005d8bffce"
 					(reference "#PWR016")
@@
 		(instances
 			(project "ramn"
-				(path "/5c9d0d4a-249f-45d4-a492-4d8f074d1b1c"
-					(reference "C?")
-					(unit 1)
-				)
 				(path "/5c9d0d4a-249f-45d4-a492-4d8f074d1b1c/00000000-0000-0000-0000-00005d8bffce"
 					(reference "C7")
@@
 		(instances
 			(project "ramn"
-				(path "/5c9d0d4a-249f-45d4-a492-4d8f074d1b1c"
-					(reference "C?")
-					(unit 1)
-				)
 				(path "/5c9d0d4a-249f-45d4-a492-4d8f074d1b1c/00000000-0000-0000-0000-00005d8bffce"
 					(reference "C8")
@@
 		(instances
 			(project "ramn"
-				(path "/5c9d0d4a-249f-45d4-a492-4d8f074d1b1c"
-					(reference "#PWR?")
-					(unit 1)
-				)
 				(path "/5c9d0d4a-249f-45d4-a492-4d8f074d1b1c/00000000-0000-0000-0000-00005d8bffce"
 					(reference "#PWR017")
@@
 		(instances
 			(project "ramn"
-				(path "/5c9d0d4a-249f-45d4-a492-4d8f074d1b1c"
-					(reference "#PWR?")
-					(unit 1)
-				)
 				(path "/5c9d0d4a-249f-45d4-a492-4d8f074d1b1c/00000000-0000-0000-0000-00005d8bffce"
 					(reference "#PWR020")
@@
 		(instances
 			(project "ramn"
-				(path "/5c9d0d4a-249f-45d4-a492-4d8f074d1b1c"
-					(reference "Y?")
-					(unit 1)
-				)
 				(path "/5c9d0d4a-249f-45d4-a492-4d8f074d1b1c/00000000-0000-0000-0000-00005d8bffce"
 					(reference "Y1")
@@
 		(instances
 			(project "ramn"
-				(path "/5c9d0d4a-249f-45d4-a492-4d8f074d1b1c"
-					(reference "C?")
-					(unit 1)
-				)
 				(path "/5c9d0d4a-249f-45d4-a492-4d8f074d1b1c/00000000-0000-0000-0000-00005d8bffce"
 					(reference "C5")
@@
 		(instances
 			(project "ramn"
-				(path "/5c9d0d4a-249f-45d4-a492-4d8f074d1b1c"
-					(reference "C?")
-					(unit 1)
-				)
 				(path "/5c9d0d4a-249f-45d4-a492-4d8f074d1b1c/00000000-0000-0000-0000-00005d8bffce"
 					(reference "C6")
@@
 		(instances
 			(project "ramn"
-				(path "/5c9d0d4a-249f-45d4-a492-4d8f074d1b1c"
-					(reference "#PWR?")
-					(unit 1)
-				)
 				(path "/5c9d0d4a-249f-45d4-a492-4d8f074d1b1c/00000000-0000-0000-0000-00005d8bffce"
 					(reference "#PWR014")
@@
 		(instances
 			(project "ramn"
-				(path "/5c9d0d4a-249f-45d4-a492-4d8f074d1b1c"
-					(reference "#PWR?")
-					(unit 1)
-				)
 				(path "/5c9d0d4a-249f-45d4-a492-4d8f074d1b1c/00000000-0000-0000-0000-00005d8bffce"
 					(reference "#PWR013")
@@
 		(instances
 			(project "ramn"
-				(path "/5c9d0d4a-249f-45d4-a492-4d8f074d1b1c"
-					(reference "BOOT?")
-					(unit 1)
-				)
 				(path "/5c9d0d4a-249f-45d4-a492-4d8f074d1b1c/00000000-0000-0000-0000-00005d8bffce"
 					(reference "BOOT0")
@@
 		(instances
 			(project "ramn"
-				(path "/5c9d0d4a-249f-45d4-a492-4d8f074d1b1c/00000000-0000-0000-0000-00005d815e09"
-					(reference "J?")
-					(unit 1)
-				)
 				(path "/5c9d0d4a-249f-45d4-a492-4d8f074d1b1c/00000000-0000-0000-0000-00005d8bffce"
 					(reference "J3")
-					(unit 1)
-				)
-				(path "/5c9d0d4a-249f-45d4-a492-4d8f074d1b1c/00000000-0000-0000-0000-00005d8ede42"
-					(reference "J?")
 					(unit 1)
 				)
@@
 		(instances
 			(project "ramn"
-				(path "/5c9d0d4a-249f-45d4-a492-4d8f074d1b1c"
-					(reference "C?")
-					(unit 1)
-				)
 				(path "/5c9d0d4a-249f-45d4-a492-4d8f074d1b1c/00000000-0000-0000-0000-00005d8bffce"
 					(reference "C3")
@@
 		(instances
 			(project "ramn"
-				(path "/5c9d0d4a-249f-45d4-a492-4d8f074d1b1c"
-					(reference "#PWR?")
-					(unit 1)
-				)
 				(path "/5c9d0d4a-249f-45d4-a492-4d8f074d1b1c/00000000-0000-0000-0000-00005d8bffce"
 					(reference "#PWR06")
@@
 		(instances
 			(project "ramn"
-				(path "/5c9d0d4a-249f-45d4-a492-4d8f074d1b1c"
-					(reference "C?")
-					(unit 1)
-				)
 				(path "/5c9d0d4a-249f-45d4-a492-4d8f074d1b1c/00000000-0000-0000-0000-00005d8bffce"
 					(reference "C4")
@@
 		(instances
 			(project "ramn"
-				(path "/5c9d0d4a-249f-45d4-a492-4d8f074d1b1c"
-					(reference "#PWR?")
-					(unit 1)
-				)
 				(path "/5c9d0d4a-249f-45d4-a492-4d8f074d1b1c/00000000-0000-0000-0000-00005d8bffce"
 					(reference "#PWR010")
@@
 		(instances
 			(project "ramn"
-				(path "/5c9d0d4a-249f-45d4-a492-4d8f074d1b1c"
-					(reference "#PWR?")
-					(unit 1)
-				)
 				(path "/5c9d0d4a-249f-45d4-a492-4d8f074d1b1c/00000000-0000-0000-0000-00005d8bffce"
 					(reference "#PWR09")
@@
 		(on_board yes)
 		(in_pos_files yes)
-		(dnp no)
+		(dnp yes)
 		(property "Reference" "R9"
 			(at 173.99 100.33 0)
@@
 		(instances
 			(project "ramn"
-				(path "/5c9d0d4a-249f-45d4-a492-4d8f074d1b1c"
-					(reference "R?")
-					(unit 1)
-				)
-				(path "/5c9d0d4a-249f-45d4-a492-4d8f074d1b1c/00000000-0000-0000-0000-00005d815e09"
-					(reference "R?")
-					(unit 1)
-				)
 				(path "/5c9d0d4a-249f-45d4-a492-4d8f074d1b1c/00000000-0000-0000-0000-00005d8bffce"
 					(reference "R9")
-					(unit 1)
-				)
-				(path "/5c9d0d4a-249f-45d4-a492-4d8f074d1b1c/00000000-0000-0000-0000-00005d8ede42"
-					(reference "R?")
 					(unit 1)
 				)
@@
 		(instances
 			(project "ramn"
-				(path "/5c9d0d4a-249f-45d4-a492-4d8f074d1b1c"
-					(reference "#PWR?")
-					(unit 1)
-				)
 				(path "/5c9d0d4a-249f-45d4-a492-4d8f074d1b1c/00000000-0000-0000-0000-00005d8bffce"
 					(reference "#PWR015")
@@
 		(instances
 			(project "ramn"
-				(path "/5c9d0d4a-249f-45d4-a492-4d8f074d1b1c"
-					(reference "R?")
-					(unit 1)
-				)
-				(path "/5c9d0d4a-249f-45d4-a492-4d8f074d1b1c/00000000-0000-0000-0000-00005d815e09"
-					(reference "R?")
-					(unit 1)
-				)
 				(path "/5c9d0d4a-249f-45d4-a492-4d8f074d1b1c/00000000-0000-0000-0000-00005d8bffce"
 					(reference "R8")
 					(unit 1)
 				)
-				(path "/5c9d0d4a-249f-45d4-a492-4d8f074d1b1c/00000000-0000-0000-0000-00005d8ede42"
-					(reference "R?")
-					(unit 1)
-				)

Commit message: Feat(Hw): UpdateKiCadProjectAndStandardizeComponentProperties
Parts:
- BOOT0: value (none) -> ~; Category (none) -> Electronic Components / Switches; LCSC# C5277086 -> (none); lcsc# (none) -> C5277086; manf# (none) -> RH-5000
- C10, C3, C4, C8, C9: Category (none) -> Electronic Components / Capacitors; LCSC# C599645 -> (none); lcsc# (none) -> C599645; manf# (none) -> C0603C104J3RAC7867
- C5, C6: Category (none) -> Electronic Components / Capacitors; LCSC# C9807 -> (none); lcsc# (none) -> C9807; manf# (none) -> CL31A106KAHNNNE
- C7: Category (none) -> Electronic Components / Capacitors; LCSC# C1848 -> (none); lcsc# (none) -> C1848; manf# (none) -> CL31B105KBHNNNE
- J3: value (none) -> ~; Category (none) -> Electronic Components / Connectors; LCSC# C2897414 -> (none); lcsc# (none) -> C2897414; manf# (none) -> PM254-2-13-Z-8.5
- R8: Category (none) -> Electronic Components / Resistors; LCSC# C98220 -> (none); lcsc# (none) -> C98220; manf# (none) -> RC0603FR-0710KL
- R9: Category (none) -> Electronic Components / Resistors
- U1: Category (none) -> Electronic Components / Integrated Circuits; LCSC# C124015 -> (none); lcsc# (none) -> C124015; manf# (none) -> MCP2558FD-H/SN
- U2: Category (none) -> Electronic Components / Integrated Circuits; LCSC# C2969980 -> (none); lcsc# (none) -> C2969980; manf# (none) -> STM32L552CET6
- Y1: Category (none) -> Electronic Components / Crystals & Oscillators; LCSC# C889706 -> (none); lcsc# (none) -> C889706; manf# (none) -> NX3225GD-8MHZ-STD-CRA-3
