File: hardware/V1_revB/0_ramn/vanilla_uc.kicad_sch (KiCad schematic)
At the start: 14 parts, among them J4 , U4 ATA6561-GAQW-N

Commit message: Feat(Hw):Modify_BOM_LCSC#
Parts:
- C13, C14, C18, C19, C20: renamed from C?; LCSC# (none) -> C599645
- C15, C16: renamed from C?; LCSC# (none) -> C9807
- C17: renamed from C?; LCSC# (none) -> C1848
- J4: value (none) -> (none); LCSC# (none) -> C2897414
- R10, R11: renamed from R?; LCSC# (none) -> C98220
- U4: LCSC# (none) -> C124015
- U5: renamed from U?; LCSC# (none) -> C2969980
- Y2: renamed from Y?; LCSC# (none) -> C889706

Commit message: Feat(Hw): UpdateKiCadProjectAndStandardizeComponentProperties
Parts:
- C13, C14, C18, C19, C20: Category (none) -> Electronic Components / Capacitors; LCSC# C599645 -> (none); lcsc# (none) -> C599645; manf# (none) -> C0603C104J3RAC7867
- C15, C16: Category (none) -> Electronic Components / Capacitors; LCSC# C9807 -> (none); lcsc# (none) -> C9807; manf# (none) -> CL31A106KAHNNNE
- C17: Category (none) -> Electronic Components / Capacitors; LCSC# C1848 -> (none); lcsc# (none) -> C1848; manf# (none) -> CL31B105KBHNNNE
- J4: value (none) -> ~; Category (none) -> Electronic Components / Connectors; LCSC# C2897414 -> (none); lcsc# (none) -> C2897414; manf# (none) -> PM254-2-13-Z-8.5
- R10, R11: Category (none) -> Electronic Components / Resistors; LCSC# C98220 -> (none); lcsc# (none) -> C98220; manf# (none) -> RC0603FR-0710KL
- U4: Category (none) -> Electronic Components / Integrated Circuits; LCSC# C124015 -> (none); lcsc# (none) -> C124015; manf# (none) -> MCP2558FD-H/SN
- U5: Category (none) -> Electronic Components / Integrated Circuits; LCSC# C2969980 -> (none); lcsc# (none) -> C2969980; manf# (none) -> STM32L552CET6
- Y2: Category (none) -> Electronic Components / Crystals & Oscillators; LCSC# C889706 -> (none); lcsc# (none) -> C889706; manf# (none) -> NX3225GD-8MHZ-STD-CRA-3
