File: hardware/V1_revB/3_powertrain/powertrain.kicad_sch (KiCad schematic)
At the start: 25 parts, among them J6 , SW1 SKRHADE010

Commit message: Feat(Hw):Modify_BOM_LCSC#
Parts:
- 3V3, ACCEL1, BRAKE1, GND1, SHIFT1: LCSC (none) -> C5277086
- C2, C3: LCSC (none) -> C282519
- J6: value (none) -> (none); LCSC (none) -> C2897414
- R1, R2, R3, R4, R5, R6: LCSC (none) -> C209220
- RV1, RV2: LCSC (none) -> C470417
- SW1: LCSC (none) -> C202415
- TVS1, TVS2, TVS3: LCSC (none) -> C1849694

Commit message: Feat(Hw): Modify_and_fix_footprints_and_symbols
Parts:
- removed RV1, RV2: R_POT_TRIM_US, custom:RS15111A900B, symbol Device:R_POT_TRIM_US
- removed SW1: SKRHADE010, SKRHADE010, symbol custom:SKRHADE010
- added RV1, RV2: R_Potentiometer_US, RAMN_New_Footprint:RS15111A900B, symbol Device:R_Potentiometer_US
- added SW1: (no value), RAMN_New_Footprint:SKRHADE010, symbol RAMN_New_Symbols:Joystick_6P
- FID1, FID2, FID3, H1, H2: now not fitted
Connections:
- net 3V3_ECU: now also RV1.1, RV2.1
- net Accel: now also RV1.2
- net Brake: now also RV2.2
- net GND: now also RV1.3, RV2.3, SW1.5 (GND)
- net JOYSTICK: now also SW1.1 (A)
- net CENTER: now reaches R2.2, R3.1
- net CENTER: now also SW1.2 (CENTER)
- net C: now reaches R3.2, R4.1
- net C: now also SW1.3 (C)
- net at R4.2, R5.1: now also SW1.4 (B)
- net at R5.2, R6.1: now also SW1.6 (D)

Commit message: Feat(Hw): EnhanceComponentLibraries
Parts:
- 3V3, ACCEL1, BRAKE1, GND1, SHIFT1: Category (none) -> Electronic Components / Other Components; LCSC C5277086 -> (none); lcsc# (none) -> C5277086; manf# (none) -> RH-5000
- C2, C3: Category (none) -> Electronic Components / Capacitors; LCSC C282519 -> (none); lcsc# (none) -> C282519; manf# (none) -> TCC0603X7R104K500CT
- FID1, FID2, FID3: Category (none) -> Electronic Components / Other Components
- H1, H2: Category (none) -> Production & Packaging / Screws & Hardware
- J6: value (none) -> ~; Category (none) -> Electronic Components / Connectors; LCSC C2897414 -> (none); lcsc# (none) -> C2897414; manf# (none) -> PM254-2-13-Z-8.5
- R1, R2, R3, R4, R5, R6: Category (none) -> Electronic Components / Resistors; LCSC C209220 -> (none); lcsc# (none) -> C209220; manf# (none) -> RMS06JT103
- RV1, RV2: Category (none) -> Electronic Components / Resistors; LCSC C470417 -> (none); lcsc# (none) -> C470417; manf# (none) -> RS15111A900B
- SW1: value (none) -> ~; Category (none) -> Electronic Components / Switches; LCSC C202415 -> (none); lcsc# (none) -> C202415; manf# (none) -> SKRHADE010
- TVS1, TVS2, TVS3: Category (none) -> Electronic Components / Other Components; LCSC C1849694 -> (none); lcsc# (none) -> C1849694; manf# (none) -> SMF5V0TR
