File: hardware/V1_revB/3_powertrain/powertrain.kicad_pcb (KiCad board)
At the start: 2 copper layers, 39.1 x 44.7 mm, 25 parts, among them J6 , SW1 SKRHADE010

Commit message: Feat(Hw): Modify_and_fix_footprints_and_symbols
Parts:
- J6: value (none) -> ~
- RV1, RV2: value R_POT_TRIM_US -> R_Potentiometer_US; footprint custom:RS15111A900B -> RAMN_New_Footprint:RS15111A900B
- SW1: value SKRHADE010 -> ~; footprint custom:SKRHADE010 -> RAMN_New_Footprint:SKRHADE010
Connections:
- net Net-(R2-Pad2) renamed /CENTER
- net Net-(R3-Pad2) renamed /C
Routing:
- net GND: track 0.00 -> 8.38 mm
- net Net-(SW1-B): track 13.9 -> 12.7 mm

Commit message: Feat(Hw): UpdatePCBsToV1.2Revision
Other:
- board text added: "RAMN V1.2"
- board text removed: "RAMN"
Changed lines of the file:
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@@
 		(layer "Edge.Cuts")
 	)
-	(gr_text "RAMN"
+	(gr_text "RAMN V1.2"
 		(at 51.308 25.146 0)
 		(layer "B.Cu")
