File: hardware/V1_revB/4_body/body.kicad_sch (KiCad schematic)
At the start: 28 parts, among them SW4 SK14EG13, U1 STP08CP05XT

Commit message: Feat(Hw):Modify_BOM_LCSC#
Parts:
- C1: LCSC (none) -> C282519
- D1, D2, D6: LCSC (none) -> C51933295
- D3, D4, D5: LCSC (none) -> C510294
- D7: LCSC (none) -> C19273153
- D8: LCSC (none) -> C51933292
- GND1, LE1, MOSI1, OE1, POS1, SCK1: LCSC (none) -> C5277086
- J8: value ~ -> (none); LCSC (none) -> C2897414
- R12, R13, R14: LCSC (none) -> C209220
- R15: LCSC (none) -> C171725
- SW4: LCSC (none) -> C34362858
- TVS7: LCSC (none) -> C1849694
- U1: LCSC (none) -> C2678539

Commit message: Feat(Hw): Modify_and_fix_footprints_and_symbols
Parts:
- removed SW4: SK14EG13, custom:SK14EG13, symbol custom:SK14EG13
- added SW2: (no value), RAMN_New_Footprint:SK14dG13, symbol RAMN_New_Symbols:SK14DG13
- FID1, FID2, FID3, H5, H6: now not fitted
Connections:
- net 3V3_ECU: now also SW2.3 (3V3)
- net GND: now also SW2.1 (GND)
- net Key: now also SW2.C1 (KEY)
- net at R13.1, R14.2: now also SW2.2 (Pad1)
Other:
- moved on the sheet: POS1, TVS7

Commit message: Feat(Hw): EnhanceComponentLibraries
Parts:
- SW4: renamed from SW2; LCSC (none) -> C34362858
Changed lines of the file:
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@@
 		(dnp no)
 		(fields_autoplaced yes)
-		(property "Reference" "SW2"
+		(property "Reference" "SW4"
 			(at 167.64 91.44 0)
 			(show_name no)
@@
 			)
 		)
+		(property "LCSC" "C34362858"
+			(at 167.64 102.87 0)
+			(hide yes)
+			(show_name no)
+			(do_not_autoplace no)
+			(effects
+				(font
+					(size 1.27 1.27)
+				)
+			)
+		)
 		(pin "2"
 		)
@@
 			(project "body"
 				(path "/a57f77f6-6a96-464e-9c74-0d342c7a10ff"
-					(reference "SW2")
+					(reference "SW4")
 					(unit 1)
 				)

Commit message: Feat(Hw): UpdateKiCadProjectAndStandardizeComponentProperties
Parts:
- C1: Category (none) -> Electronic Components / Capacitors; LCSC C282519 -> (none); lcsc# (none) -> C282519; manf# (none) -> TCC0603X7R104K500CT
- D1, D2, D6: Category (none) -> Electronic Components / Diodes; LCSC C51933295 -> (none); lcsc# (none) -> C51933295; manf# (none) -> GL0603UY01
- D3, D4, D5: Category (none) -> Electronic Components / Diodes; LCSC C510294 -> (none); lcsc# (none) -> C510294; manf# (none) -> SML-E12V8WT86
- D7: Category (none) -> Electronic Components / Diodes; LCSC C19273153 -> (none); lcsc# (none) -> C19273153; manf# (none) -> YLED0603O
- D8: Category (none) -> Electronic Components / Diodes; LCSC C51933292 -> (none); lcsc# (none) -> C51933292; manf# (none) -> GL0603UR01
- FID1, FID2, FID3: Category (none) -> Electronic Components / Other Components
- GND1, LE1, MOSI1, OE1, POS1, SCK1: Category (none) -> Electronic Components / Other Components; LCSC C5277086 -> (none); lcsc# (none) -> C5277086; manf# (none) -> RH-5000
- H5, H6: Category (none) -> Production & Packaging / Screws & Hardware
- J8: value (none) -> ~; Category (none) -> Electronic Components / Connectors; LCSC C2897414 -> (none); lcsc# (none) -> C2897414; manf# (none) -> PM254-2-13-Z-8.5
- R12, R13, R14: Category (none) -> Electronic Components / Resistors; LCSC C209220 -> (none); lcsc# (none) -> C209220; manf# (none) -> RMS06JT103
- R15: Category (none) -> Electronic Components / Resistors; LCSC C171725 -> (none); lcsc# (none) -> C171725; manf# (none) -> RK73B1JTTD182J
- SW4: value (none) -> ~; Category (none) -> Electronic Components / Switches; LCSC C34362858 -> (none); lcsc# (none) -> C34362858; manf# (none) -> SK14DG13
- TVS7: Category (none) -> Electronic Components / Other Components; LCSC C1849694 -> (none); lcsc# (none) -> C1849694; manf# (none) -> SMF5V0TR
- U1: Category (none) -> Electronic Components / Integrated Circuits; LCSC C2678539 -> (none); lcsc# (none) -> C2678539; manf# (none) -> STP08CP05TTR
