File: hardware/V1_revB/4_body/body.kicad_pcb (KiCad board)
At the start: 2 copper layers, 57.8 x 40.6 mm, 36 parts, among them SW4 SK14EG13, U1 STP08CP05XT

Commit message: Feat(Hw): Modify_and_fix_footprints_and_symbols
Parts:
- removed SW4: SK14EG13, custom:SK14EG13
- added SW2: ~, RAMN_New_Footprint:SK14dG13, F.Cu at (40.8, 36.4)
Routing:
- net GND: track 23.9 -> 28.4 mm

Commit message: Feat(Hw): EnhanceComponentLibraries
Parts:
- renumbered SW2 to SW4
Changed lines of the file:
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@@
 		(layer "F.Cu")
 		(at 40.767 36.449)
-		(property "Reference" "SW2"
+		(property "Reference" "SW4"
 			(at -2.286 8.636 180)
 			(layer "F.SilkS")
@@
 					(thickness 0.15)
 				)
+			)
+		)
+		(property "LCSC" "C34362858"
+			(at 0 0 0)
+			(unlocked yes)
+			(layer "F.Fab")
+			(hide yes)
+			(effects
+				(font
+					(size 1 1)
+					(thickness 0.15)
+				)

Commit message: Feat(Hw): UpdatePCBsToV1.2Revision
Other:
- board text added: "RAMN V1.2"
- board text removed: "RAMN"
Changed lines of the file:
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@@
 		(layer "Edge.Cuts")
 	)
-	(gr_text "RAMN"
-		(at 64.262 40.386 0)
+	(gr_text "RAMN V1.2"
+		(at 66.03 42.24 0)
 		(layer "B.Cu")
 		(effects
