File: hardware/V1_revB/5_debugger/debugger.kicad_sch (KiCad schematic)
At the start: 29 parts, among them J10 Conn_ARM_JTAG_SWD_20

Commit message: Feat(Hw):Modify_BOM_LCSC#
Parts:
- 3V3, 5V1, GND1, GND2, JTCK1, JTDI1, JTDO1, JTMS1, JTRST1, PA1, PA2, PA3, PA4, PA5, PA6, PA7, PA8, PB0, PB1, PB10, PB11, PB12, PB13, PB14, PB15, PB2, nRST1: LCSC (none) -> C5277086
- J10: LCSC (none) -> C7527716
- J9: value ~ -> (none); LCSC (none) -> C2897414

Commit message: Feat(Hw): UpdateKiCadProjectAndStandardizeComponentProperties
Parts:
- 3V3, 5V1, GND1, GND2, JTCK1, JTDI1, JTDO1, JTMS1, JTRST1, PA1, PA2, PA3, PA4, PA5, PA6, PA7, PA8, PB0, PB1, PB10, PB11, PB12, PB13, PB14, PB15, PB2, nRST1: Category (none) -> Electronic Components / Other Components; LCSC C5277086 -> (none); lcsc# (none) -> C5277086; manf# (none) -> RH-5000
- J10: Category (none) -> Electronic Components / Connectors; LCSC C7527716 -> (none); lcsc# (none) -> C7527716; manf# (none) -> XDFH-0259-2*10P
- J9: value (none) -> ~; Category (none) -> Electronic Components / Connectors; LCSC C2897414 -> (none); lcsc# (none) -> C2897414; manf# (none) -> PM254-2-13-Z-8.5
